File: schematic_pcb/RoboArm/RoboArm.kicad_sch (KiCad schematic)
At the start: 36 parts, among them M1 Motor_Servo, M2 Motor_Servo, M3 Motor_Servo, M4 Motor_Servo, M5 Motor_Servo, M6 Motor_Servo, M7 Motor_Servo, M8 Motor_Servo, M9 Motor_Servo, U1 ESP32-DEVKIT-V1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

Commit message: updated july 29th and 30th
Parts:
- removed Dynamixel XM1: ~, symbol Dynamixel:Dynamixel_XM430_W350
- removed Dynamixel XM2: ~, symbol Dynamixel:Dynamixel_XM430_W350
- removed Dynamixel XM3: ~, symbol Dynamixel:Dynamixel_XM430_W350
- removed Dynamixel XM4: ~, symbol Dynamixel:Dynamixel_XM430_W350
- added LX-255_Servo_Motor1, LX-255_Servo_Motor2, LX-255_Servo_Motor3, LX-255_Servo_Motor4: ~, symbol LX-255 Servo:LX-255_Servo_Motor
- added U10: LM2596S-ADJ, Package_TO_SOT_SMD:TO-263-5_TabPin3, symbol Regulator_Switching:LM2596S-ADJ
Connections:
- net +5V: now also LX-255_Servo_Motor1.2 (VCC), LX-255_Servo_Motor2.2 (VCC), LX-255_Servo_Motor3.2 (VCC), LX-255_Servo_Motor4.2 (VCC)
- net GND: now also LX-255_Servo_Motor1.1 (GND), LX-255_Servo_Motor2.1 (GND), LX-255_Servo_Motor3.1 (GND), LX-255_Servo_Motor4.1 (GND), U10.3 (GND)
- net at U8.20 (B1): now also LX-255_Servo_Motor1.3 (DATA)
- net at U8.18 (B2): now also LX-255_Servo_Motor2.3 (DATA)
- net at U8.17 (B3): now also LX-255_Servo_Motor3.3 (DATA)
- net at U8.16 (B4): now also LX-255_Servo_Motor4.3 (DATA)
- new net +7.5V: U10.1 (VIN)
- no-connect marks 52 -> 55
